Commit message: Derive the finger joint from the linkage geometry instead of two guessed anchors
The width-to-joint mapping ran linearly between `angle_open` 0.0 and
`angle_closed` 0.6. Neither anchor was a real end of travel, and the
result was visible in the planning model: "fully open" put the pads
93.8 mm apart instead of 160 mm, and "fully closed" left a 4.8 mm gap.
The modelled hand therefore reached into every object wider than 94 mm
and never quite shut. move_group checks this same URDF, so at equal
commanded width the modelled gripper was NARROWER than the real one --
every clearance check around the hand was optimistic.

The linkage itself is fine and is an RG6. From the joint origins in
onrobot_rg6_model_macro.xacro the two inner_finger origins sit

    d(q) = 2 * (0.024112 + 0.080 * cos(q + 0.93757))

apart, so the upper joint limit (+0.628319) IS the zero-width pose and
the crank dead point (-0.93757) gives 159.0 mm of clear width -- the
RG6's stroke. Only the sub-range the width was mapped onto was wrong.

`rg6_control::linkage` now carries that relation, and the sim node, the
real driver and the tool-data broadcaster all use it. The broadcaster
keeps voltage->width linear (that is the hardware's characteristic) and
puts the kinematics after it, instead of folding both into one line. The
open-side joint limit moves to the dead point so the full width is
representable at all, and the SRDF group states "open"/"close" follow.

Measured on the husky-offboard container 2026-08-16, three independent
ways: the algebra above; TF between rg6_left_inner_finger and
rg6_right_inner_finger (143 / 112 / 80 / 54 mm at commanded
160 / 100 / 45 / 0 mm); and move_group's own check_state_validity
against a widening box between the pads (92 / 60 / 28 / 4 mm).

STATUS -- do not merge yet. The 12 unit tests pass and the rebuilt sim
node starts at -0.9375699, i.e. genuinely open, which the old build could
not. But a gripper COMMAND still lands in the node with a different width
than was sent (100 mm arrives as 62.3 mm), so the command path still
renders the old numbers. That is a second defect, between the twin client
and the node, and it is not this change. It has to be found before this
branch is worth merging. The real gripper has not been measured at all --
see R19 in the workspace's ROBOTER-TODO.

File: rg6/src/rg6_description/urdf/onrobot_rg6_model_macro.xacro (robot description, xacro)
@@ -108,5 +108,5 @@
       <child link="${prefix}${fingerprefix}_inner_knuckle" />
       <axis xyz="1 0 0" />
-      <limit lower="-0.628319" upper="0.628319" velocity="2.0" effort="1000" />
+      <limit lower="-0.937570" upper="0.628319" velocity="2.0" effort="1000" />
       <mimic joint="${prefix}finger_joint" multiplier="-1" offset="0" />
     </joint>
@@ -118,9 +118,21 @@
       <child link="${prefix}${fingerprefix}_inner_finger" />
       <axis xyz="1 0 0" />
-      <limit lower="-0.872665" upper="0.872665" velocity="2.0" effort="1000" />
+      <limit lower="-0.937570" upper="0.872665" velocity="2.0" effort="1000" />
       <mimic joint="${prefix}finger_joint" multiplier="1" offset="0" />
     </joint>
   </xacro:macro>
   <xacro:include filename="$(find rg6_description)/urdf/onrobot_rg6.xacro" />
+  <!-- GELENKGRENZEN, offene Seite (2026-08-16).
+       Die untere Grenze lag symmetrisch bei -0.628319 (+-36 Grad). Die
+       Kinematik dieses Getriebes gibt aber mehr her: der Abstand der beiden
+       inner_finger-Ursprunge ist 2*(0.024112 + 0.080*cos(q + 0.93757)), also
+       maximal bei q = -0.93757 (Kurbel-Totlage). Dort betraegt die lichte
+       Weite zwischen den Pads 159,0 mm -- der Hub eines RG6. Bei -0.628319
+       waren es 151,4 mm, bei q = 0 (dem frueheren "offen") nur 93,8 mm.
+       Die Grenze wird deshalb auf die Totlage gelegt, damit die volle Weite
+       ueberhaupt darstellbar ist; die geschlossene Seite bleibt, sie sitzt
+       bereits auf der Stellung mit Weite null.
+       Am husky-offboard-Container per TF und per check_state_validity
+       nachgemessen; die Gegenprobe an der echten Hand steht aus (R19). -->
   <xacro:macro name="finger_joint" params="prefix">
     <joint name="${prefix}finger_joint" type="revolute">
@@ -129,5 +141,5 @@
       <child link="${prefix}left_outer_knuckle" />
       <axis xyz="-1 0 0" />
-      <limit lower="-0.628319" upper="0.628319" velocity="2.0" effort="1000" />
+      <limit lower="-0.937570" upper="0.628319" velocity="2.0" effort="1000" />
     </joint>
     <xacro:finger_joints prefix="${prefix}" fingerprefix="left" reflect="1.0"/>
@@ -139,5 +151,5 @@
       <child link="${prefix}right_outer_knuckle" />
       <axis xyz="1 0 0" />
-      <limit lower="-0.628319" upper="0.628319" velocity="2.0" effort="1000" />
+      <limit lower="-0.937570" upper="0.628319" velocity="2.0" effort="1000" />
       <mimic joint="${prefix}finger_joint" multiplier="-1" offset="0" />
     </joint>

Commit message: Make the linkage model loadable, mirrored and self-consistent
Three defects in the previous commit on this branch, each of which would have
survived a green rg6_control test run because none of them is visible there.

The gripper description was not valid XML.  A comment carried a double hyphen,
which XML forbids, so xacro aborted on it and the whole robot model failed to
render — mock could not start at all.  The earlier test run only built
rg6_control, never rg6_description, which is why it went unnoticed.

The two joints that mimic the driver with multiplier -1 had their limit
widened on the same side as the driver's.  While both sides sat symmetrically
at +-0.628319 that was harmless; with the open side reaching further it is
not, and at the fully open pose those joints stood above their own upper
bound.  Their limits are now the mirrored ones.

Crank length and phase were pinned as literals and sat 0.09 mrad away from the
geometry they describe.  They are derived from the two offsets read off the
URDF instead, which also fixes the driver joint's lower limit: it was rounded
towards zero and therefore excluded the very pose it was meant to allow.  The
same four read-off numbers now live in the robot profile (robot_contract,
gripper.linkage), so both sides of the GripperCommand action compute from the
same source.

Measured in the husky-offboard container afterwards: commanded 160/100/45/0 mm
now stand at 159.0/100.0/45.0/0.0 mm of clear width, against 93.7/62.5/31.1/4.3
before.  TF between the two inner_finger frames reads 149 mm at 100 mm
commanded, as the geometry predicts.

File: rg6/src/rg6_description/urdf/onrobot_rg6_model_macro.xacro (robot description, xacro)
@@ -108,5 +108,9 @@
       <child link="${prefix}${fingerprefix}_inner_knuckle" />
       <axis xyz="1 0 0" />
-      <limit lower="-0.937570" upper="0.628319" velocity="2.0" effort="1000" />
+      <!-- multiplier="-1": dieses Gelenk laeuft dem Treibergelenk ENTGEGEN,
+           seine Grenzen sind also die gespiegelten.  Solange beide Seiten
+           symmetrisch bei +-0.628319 lagen, war das folgenlos; seit die offene
+           Seite weiter reicht, ist es das nicht mehr. -->
+      <limit lower="-0.628319" upper="0.937658" velocity="2.0" effort="1000" />
       <mimic joint="${prefix}finger_joint" multiplier="-1" offset="0" />
     </joint>
@@ -118,5 +122,7 @@
       <child link="${prefix}${fingerprefix}_inner_finger" />
       <axis xyz="1 0 0" />
-      <limit lower="-0.937570" upper="0.872665" velocity="2.0" effort="1000" />
+      <!-- multiplier="1": laeuft MIT dem Treibergelenk, Grenzen also wie dort
+           (die obere bleibt weiter, sie war schon vorher grosszuegig). -->
+      <limit lower="-0.937658" upper="0.872665" velocity="2.0" effort="1000" />
       <mimic joint="${prefix}finger_joint" multiplier="1" offset="0" />
     </joint>
@@ -126,11 +132,14 @@
        Die untere Grenze lag symmetrisch bei -0.628319 (+-36 Grad). Die
        Kinematik dieses Getriebes gibt aber mehr her: der Abstand der beiden
-       inner_finger-Ursprunge ist 2*(0.024112 + 0.080*cos(q + 0.93757)), also
-       maximal bei q = -0.93757 (Kurbel-Totlage). Dort betraegt die lichte
-       Weite zwischen den Pads 159,0 mm -- der Hub eines RG6. Bei -0.628319
-       waren es 151,4 mm, bei q = 0 (dem frueheren "offen") nur 93,8 mm.
+       inner_finger-Ursprunge ist 2*(0.024112 + 0.080*cos(q + 0.93766)), also
+       maximal bei q = -0.93766 (Kurbel-Totlage). Dort betraegt die lichte
+       Weite zwischen den Pads 159,0 mm - der Hub eines RG6. Bei -0.628319
+       waren es 151,4 mm, bei q = 0 (dem frueheren "offen") nur 93,7 mm.
        Die Grenze wird deshalb auf die Totlage gelegt, damit die volle Weite
        ueberhaupt darstellbar ist; die geschlossene Seite bleibt, sie sitzt
        bereits auf der Stellung mit Weite null.
+       Gerundet wird dabei VON NULL WEG: atan2(0.064495, 0.047335) ist
+       0.9376577, eine Grenze diesseits davon (der erste Anlauf hatte
+       -0.937570) macht genau die Stellung ungueltig, die "ganz offen" heisst.
        Am husky-offboard-Container per TF und per check_state_validity
        nachgemessen; die Gegenprobe an der echten Hand steht aus (R19). -->
@@ -141,5 +150,5 @@
       <child link="${prefix}left_outer_knuckle" />
       <axis xyz="-1 0 0" />
-      <limit lower="-0.937570" upper="0.628319" velocity="2.0" effort="1000" />
+      <limit lower="-0.937658" upper="0.628319" velocity="2.0" effort="1000" />
     </joint>
     <xacro:finger_joints prefix="${prefix}" fingerprefix="left" reflect="1.0"/>
@@ -151,5 +160,6 @@
       <child link="${prefix}right_outer_knuckle" />
       <axis xyz="1 0 0" />
-      <limit lower="-0.937570" upper="0.628319" velocity="2.0" effort="1000" />
+      <!-- multiplier="-1": gespiegelte Grenzen, siehe inner_knuckle_joint. -->
+      <limit lower="-0.628319" upper="0.937658" velocity="2.0" effort="1000" />
       <mimic joint="${prefix}finger_joint" multiplier="-1" offset="0" />
     </joint>
