Commit message: Fix collision meshes

File: rg6/src/rg6_description/urdf/onrobot_rg6.xacro (robot description, xacro)
@@ -17,26 +17,22 @@
         </material>
       </visual>
-      <!-- ZWEI enge Huell-Boxen fuer den GANZEN Greifer, beide in DIESEM Link:
-           weiterhin keine Selbstkollision innerhalb des Greifers (mehrere
-           <collision>-Elemente eines Links bilden fuer MoveIt EINEN Koerper),
-           aber deutlich engere Umgebungs-/Armpruefung als die alte Einzelbox
-           0.11x0.19x0.25 (die blockierte z.B. Posen mit dem Greifer ueber dem
-           Husky-Topplate als Scheinkollision, s. hrl-Scan-Pose).
-           Masse aus den Visual-Meshes vermessen (twinlink/MuJoCo, voller
-           Fingerhub t=0..0.6), Marge ~5 mm:
-             Gehaeuse:  x[-0.036,+0.040] y[+-0.042] z[0..0.167]
-             Finger:    x[+-0.013]       y[+-0.078] z[0.121..0.283] (Hub-Union)
-           Gehaeuse-Box startet bei z=0.02 -> reicht NICHT in arm_0_wrist_3_link
-           zurueck (kein Handgelenk-Falschtreffer). -->
+      <!-- NUR NOCH die Gehaeuse-Huell-Box (Greifer-Koerper / Motorhaus) an
+           DIESEM Link. Frueher gab es zusaetzlich eine statische Finger-Huell-Box
+           (Union ueber den ganzen Fingerhub, origin 0 0 0.205, 0.036x0.166x0.170),
+           fest am base_link -> hat jeden Zugriff *zwischen* die Pads blockiert, so
+           dass Greifen im Planer unmoeglich war. Die Finger haben jetzt eigene
+           artikulierte Collision (onrobot_rg6_model_macro.xacro), die sich mit dem
+           Greifhub bewegt; die Intra-Greifer-Self-Collision wird per SRDF via
+           rg6_moveit_patch deaktiviert.
+           Gehaeuse-Masse aus den Visual-Meshes vermessen (twinlink/MuJoCo),
+           Marge ~5 mm: x[-0.036,+0.040] y[+-0.042] z[0..0.167].
+           Box startet bei z=0.02 -> reicht NICHT in arm_0_wrist_3_link zurueck
+           (kein Handgelenk-Falschtreffer). D435 (camera_0_link) sitzt auf der
+           Gehaeuse-Oberseite (robot.yaml: parent base_link, xyz 0.023/0/0.14) ->
+           base<->camera ist im SRDF 'Adjacent' deaktiviert. -->
       <collision>
         <origin xyz="0.002 0 0.095" rpy="0 0 0"/>
         <geometry>
           <box size="0.086 0.094 0.150"/>
-        </geometry>
-      </collision>
-      <collision>
-        <origin xyz="0 0 0.205" rpy="0 0 0"/>
-        <geometry>
-          <box size="0.036 0.166 0.170"/>
         </geometry>
       </collision>

File: rg6/src/rg6_description/urdf/onrobot_rg6_model_macro.xacro (robot description, xacro)
@@ -33,6 +33,17 @@
         </material>
       </visual>
-      <!-- collision bewusst weggelassen: 4-Gelenk-Schleife im URDF-Baum -> sonst
-           Selbstkollision -> MoveIt-Planung schlaegt fehl. Greifer ist Anzeige-only. -->
+      <!-- Collision = Visual-Mesh. Frueher bewusst weggelassen (4-Gelenk-Schleife
+           -> Selbstkollision -> MoveIt-Planung schlug fehl, Greifer war Anzeige-only).
+           Jetzt: echte artikulierte Collision pro Link -> Greifen im Planer moeglich.
+           Die Selbstkollision der Intra-Greifer-Paare (4-Barlenk + Kamera + wrist_3 +
+           Fingerspitzen gegeneinander) wird per SRDF <disable_collisions> deaktiviert,
+           geschrieben vom rg6_moveit_patch (Marker 'collision-disable') NACH jedem
+           moveit_collision_updater-Lauf. Greifer prueft weiter gegen Welt/Arm. -->
+      <collision>
+        <origin xyz="0 0 0" rpy="0 0 0" />
+        <geometry>
+          <mesh filename="package://rg6_description/meshes/visual/outer_knuckle.stl" />
+        </geometry>
+      </collision>
     </link>
   </xacro:macro>
@@ -53,5 +64,12 @@
         </material>
       </visual>
-      <!-- collision weggelassen (siehe outer_knuckle). -->
+      <!-- collision: Visual-Mesh (siehe outer_knuckle); Intra-Greifer-Self-Collision
+           per SRDF via rg6_moveit_patch deaktiviert. -->
+      <collision>
+        <origin xyz="0 0 0" rpy="0 0 0" />
+        <geometry>
+          <mesh filename="package://rg6_description/meshes/visual/inner_knuckle.stl" />
+        </geometry>
+      </collision>
     </link>
   </xacro:macro>
@@ -72,5 +90,14 @@
         </material>
       </visual>
-      <!-- collision weggelassen (siehe outer_knuckle). -->
+      <!-- collision: Visual-Mesh. Dies sind die Greif-Pads (Kontaktflaeche zum
+           Objekt). Intra-Greifer-Self-Collision (inkl. link<->right Pads gegeneinander)
+           per SRDF via rg6_moveit_patch deaktiviert -> MoveIt kann close ohne
+           Self-Collision-Abbruch planen; rg6_control stoppt kraftgeregelt am Objekt. -->
+      <collision>
+        <origin xyz="0 0 0" rpy="0 0 0" />
+        <geometry>
+          <mesh filename="package://rg6_description/meshes/visual/inner_finger.stl" />
+        </geometry>
+      </collision>
     </link>
   </xacro:macro>

Commit message: Give the gripper the mass and centre of gravity its datasheet states
The model weighed 1.00 kg: 0.7 kg on the housing plus six 0.05 kg finger
links.  The RG6 datasheet (manual v6.6.2 DE, section 8.3.2) says 1.25 kg with
its centre of gravity 90 mm above the tool base point, and the model put that
centre at the origin.  250 g and 90 mm of lever arm are not nothing for an
end effector: MoveIt ignores inertia, but the MuJoCo twin does not, and the
number a person reads off the model to set the arm's payload was wrong.

The housing now carries the remainder that makes the assembly total 1.25 kg,
and its inertial origin sits where the whole assembly's centre of gravity
lands on the datasheet's 90 mm at half stroke.  Over the full stroke it runs
between 85.5 and 91.9 mm, because the fingers swing forward as they close and
the datasheet gives only one number.

The inertia tensor stays the placeholder it always was — the same value for a
0.05 kg jaw and a 0.95 kg housing cannot be right, but measuring it is its own
piece of work and not part of this fix.

File: rg6/src/rg6_description/urdf/onrobot_rg6.xacro (robot description, xacro)
@@ -3,7 +3,25 @@
   <xacro:macro name="onrobot_rg6_base_link" params="prefix">
     <link name="${prefix}onrobot_rg6_base_link">
+      <!-- MASSE UND SCHWERPUNKT nach Datenblatt (OnRobot RG6,
+           Bedienungsanleitung v6.6.2 DE, Abschnitt 8.3.2: 1,25 kg,
+           Schwerpunkt cZ = 90 mm vom Werkzeug-Basispunkt).
+           Vorher wog das Modell 1,00 kg: 0,7 kg hier plus 6 x 0,05 kg auf den
+           Fingergliedern - 250 g zu leicht, und der Schwerpunkt sass im
+           Ursprung statt 90 mm darueber.  Die 0,95 kg hier sind der Rest, der
+           mit den sechs Fingergliedern zusammen die 1,25 kg des Datenblatts
+           ergibt; die 0,0669 m sind so gewaehlt, dass der Schwerpunkt der
+           GANZEN Baugruppe bei halbem Hub auf den 90 mm des Datenblatts
+           landet.  Ueber den vollen Hub wandert er zwischen 85,5 und 91,9 mm,
+           weil die Finger beim Schliessen nach vorn schwingen - das
+           Datenblatt gibt nur eine Zahl, also ist die Mittelstellung der
+           ehrlichste Bezugspunkt.
+           Der Traegheitstensor bleibt der Platzhalter, der er war (fuer eine
+           0,05-kg-Backe und ein 0,95-kg-Gehaeuse derselbe Wert - das kann
+           nicht stimmen).  Fuer MoveIt ist er ohne Bedeutung, fuer MuJoCo
+           waere er es nicht; ihn zu vermessen ist eigene Arbeit und nicht
+           Teil dieses Fixes. -->
       <inertial>
-        <origin xyz="0.0 0.0 0.0" rpy="0 0 0" />
-        <mass value="0.7" />
+        <origin xyz="0.0 0.0 0.0669" rpy="0 0 0" />
+        <mass value="0.95" />
         <inertia ixx="1.0E-03" ixy="1.0E-06" ixz="1.0E-06" iyy="1.0E-03" iyz="1.0E-06" izz="1.0E-03" />
       </inertial>
