Commit message: Fix mimic behavior in viz

File: rg6/src/rg6_description/urdf/clearpath_extras.urdf.xacro (robot description, xacro)
@@ -13,7 +13,10 @@
     Sauber artikuliertes RG6 aus package 'rg6_description' (Robotiq-Stil:
     outer_knuckle/inner_knuckle/inner_finger pro Seite). Treibergelenk =
-    'rg6_finger_joint' (Praefix 'rg6_'): 0 = offen, positiv = zu. Der
-    rg6_joint_state_broadcaster setzt ALLE 6 Greifergelenke EXPLIZIT (kein
-    <mimic> - das loesen manche URDF-Parser/Foxglove nicht zuverlaessig auf).
+    'rg6_finger_joint' (Praefix 'rg6_'): 0 = offen, positiv = zu. Die 5
+    Folgegelenke haengen per <mimic> (offizielle OnRobot-Multiplier) am
+    Treibergelenk -> MoveIt animiert sie im Planungs-Preview, der ROS2
+    robot_state_publisher berechnet sie fuer /tf (Foxglove). Der
+    rg6_joint_state_broadcaster publiziert zusaetzlich alle 6 Gelenke explizit
+    (Fallback / Live-Tuning des AI2-Mappings); Werte identisch zu <mimic>.
     Kollision = eine grobe Box am base_link (keine Selbstkollision in MoveIt).
   VORAUSSETZUNG: 'rg6_description' muss in einem in robot.yaml unter

File: rg6/src/rg6_description/urdf/onrobot_rg6_model_macro.xacro (robot description, xacro)
@@ -1,7 +1,20 @@
 <?xml version="1.0"?>
 <robot xmlns:xacro="http://ros.org/wiki/xacro">
-  <!-- transmission/mimic bewusst entfernt: der rg6_joint_state_broadcaster treibt
-       alle 6 Gelenke explizit. Manche URDF-Parser (z.B. Foxglove) stolpern ueber
-       <mimic>/<transmission>/leere Material-Namen -> Meshes landen im Ursprung. -->
+  <!-- <mimic> ist WIEDER DRIN (offizielle OnRobot-Multiplier, identisch zu den
+       Werten, die der rg6_joint_state_broadcaster explizit publiziert). Ohne
+       <mimic> animiert MoveIt im Planungs-Preview nur das Treibergelenk
+       rg6_finger_joint - die 5 Folgegelenke stehen naemlich im SRDF nur als
+       <passive_joint> (nicht in der gripper-Gruppe) und werden so nicht Teil
+       der Planungs-Trajektorie. Mit <mimic> (URDF) + Aufnahme in die Gruppe
+       (rg6_moveit_patch) klassifiziert MoveIt sie als mimic_joints_ und treibt
+       sie aus rg6_finger_joint ab -> saubere Vorschau von Oeffnen/Schliessen.
+       ROS2 robot_state_publisher (jazzy) wertet <mimic> ebenfalls aus, Foxglove
+       laeuft ohnehin ueber /tf vom RSP.
+       Historie: frueher hies es, <mimic> wuerde bei Foxglove "Meshes am Ursprung"
+       ausloesen. Verursacher war aber das Original-URDF mit <material name="">
+       (LEERER Materialname) - nicht <mimic>. Die leeren Namen sind laengst durch
+       rg6_silver/rg6_black ersetzt, daher ist <mimic> sicher.
+       <transmission> bleibt weg (ros2_control holt sich keine RG6-Transmision;
+       der Greifer haengt am UR-Tool-Interface, nicht am ros2_controller). -->
   <xacro:macro name="outer_knuckle" params="prefix fingerprefix">
     <link name="${prefix}${fingerprefix}_outer_knuckle">
@@ -69,4 +82,5 @@
       <axis xyz="1 0 0" />
       <limit lower="-0.628319" upper="0.628319" velocity="2.0" effort="1000" />
+      <mimic joint="${prefix}finger_joint" multiplier="-1" offset="0" />
     </joint>
   </xacro:macro>
@@ -78,4 +92,5 @@
       <axis xyz="1 0 0" />
       <limit lower="-0.872665" upper="0.872665" velocity="2.0" effort="1000" />
+      <mimic joint="${prefix}finger_joint" multiplier="1" offset="0" />
     </joint>
   </xacro:macro>
@@ -98,4 +113,5 @@
       <axis xyz="1 0 0" />
       <limit lower="-0.628319" upper="0.628319" velocity="2.0" effort="1000" />
+      <mimic joint="${prefix}finger_joint" multiplier="-1" offset="0" />
     </joint>
     <xacro:finger_joints prefix="${prefix}" fingerprefix="right" reflect="-1.0"/>

Commit message: Put the quick changer back between the flange and the gripper

File: rg6/src/rg6_description/urdf/clearpath_extras.urdf.xacro (robot description, xacro)
@@ -45,9 +45,23 @@
   <!-- Greiferbasis an den Tool-Flansch. Modell-Achse = +Z (wie altes Modell),
        daher Roll -90deg um X. Falls noch verdreht, je 90deg variieren:
-         rpy="1.5708 0 0" | rpy="0 0 1.5708" | rpy="0 0 -1.5708" -->
+         rpy="1.5708 0 0" | rpy="0 0 1.5708" | rpy="0 0 -1.5708"
+       z = 0,0196 ist die ROBOTERSEITE des Quick Changers (Variante fuer I/O,
+       QC-Datenblatt v2.0; die Standardvariante waere 0,0136).  Sie sass bis
+       2026-08-19 auf 0, der ganze Greifer stand damit 19,6 mm zu hoch am Arm.
+       Die WERKZEUGseite steckt bereits im Mesh: die untersten 20 mm von
+       base_link.stl sind die Scheibe Ø71 mm, und der Frame liegt auf der
+       Trennebene der beiden Haelften (am Mesh nachgemessen, ROBOTER-TODO R20).
+       Unabhaengig bestaetigt am fremden Modell (inria onrobot_description,
+       rg6_v2): dort reicht body.stl 19 mm unter seinen eigenen Ursprung, mit
+       Ø69,5 mm, also dieselbe Scheibe und derselbe Bezugspunkt.
+       ACHTUNG, das verschiebt eine kalibrierte Groesse: hrl setzt fuer echte
+       Hardware descend_offset = 0,065 gegen 0,045 in der Sim, ein Aufschlag
+       von 20,0 mm, der genau diesen Fehler blind bezahlt hat.  Nach dieser
+       Korrektur greift der Arm 19,6 mm ZU HOCH, bis der Aufschlag mit
+       zurueckgenommen wird.  Nicht ohne einen Griff am Geraet nachziehen. -->
   <joint name="rg6_tool0_to_base" type="fixed">
     <parent link="arm_0_tool0"/>
     <child link="rg6_onrobot_rg6_base_link"/>
-    <origin xyz="0 0 0" rpy="0 0 -1.5708"/>
+    <origin xyz="0 0 0.0196" rpy="0 0 -1.5708"/>
   </joint>
   <!-- Greifer-TCP (mittig zwischen den Fingerspitzen, grob). -->

Commit message: Put the gripper back on the flange it is actually bolted to

File: rg6/src/rg6_description/urdf/clearpath_extras.urdf.xacro (robot description, xacro)
@@ -46,22 +46,19 @@
        daher Roll -90deg um X. Falls noch verdreht, je 90deg variieren:
          rpy="1.5708 0 0" | rpy="0 0 1.5708" | rpy="0 0 -1.5708"
-       z = 0,0196 ist die ROBOTERSEITE des Quick Changers (Variante fuer I/O,
-       QC-Datenblatt v2.0; die Standardvariante waere 0,0136).  Sie sass bis
-       2026-08-19 auf 0, der ganze Greifer stand damit 19,6 mm zu hoch am Arm.
-       Die WERKZEUGseite steckt bereits im Mesh: die untersten 20 mm von
-       base_link.stl sind die Scheibe Ø71 mm, und der Frame liegt auf der
-       Trennebene der beiden Haelften (am Mesh nachgemessen, ROBOTER-TODO R20).
-       Unabhaengig bestaetigt am fremden Modell (inria onrobot_description,
-       rg6_v2): dort reicht body.stl 19 mm unter seinen eigenen Ursprung, mit
-       Ø69,5 mm, also dieselbe Scheibe und derselbe Bezugspunkt.
-       ACHTUNG, das verschiebt eine kalibrierte Groesse: hrl setzt fuer echte
-       Hardware descend_offset = 0,065 gegen 0,045 in der Sim, ein Aufschlag
-       von 20,0 mm, der genau diesen Fehler blind bezahlt hat.  Nach dieser
-       Korrektur greift der Arm 19,6 mm ZU HOCH, bis der Aufschlag mit
-       zurueckgenommen wird.  Nicht ohne einen Griff am Geraet nachziehen. -->
+       z = 0: der Greifer sitzt UNMITTELBAR auf dem Flansch.  Am 2026-08-19
+       vom Owner am Geraet nachgesehen, nachdem hier zwischenzeitlich 0,0196
+       stand.  Diese 19,6 mm kamen aus ROBOTER-TODO R20, das aus dem
+       QC-Datenblatt geschlossen hatte, die ROBOTERSEITE des Quick Changers
+       fehle im Modell.  Der Schluss setzte eine separate QC-Scheibe zwischen
+       Flansch und Greifer voraus; die gibt es an diesem Roboter nicht.  Der
+       Fuss der Greiferbasis IST die Kopplungsflaeche (Ø71 mm, am Mesh
+       gemessen; unterste 20 mm von base_link.stl, und im fremden rg6_v2-Modell
+       ebenso als unterste Scheibe des single_bracket) und schraubt direkt auf
+       den Flansch.  Dazwischen liegt nur der 0,4-mm-Zentrierring des
+       UR-Flansches, und der ist eine Vertiefung, kein Aufbau. -->
   <joint name="rg6_tool0_to_base" type="fixed">
     <parent link="arm_0_tool0"/>
     <child link="rg6_onrobot_rg6_base_link"/>
-    <origin xyz="0 0 0.0196" rpy="0 0 -1.5708"/>
+    <origin xyz="0 0 0" rpy="0 0 -1.5708"/>
   </joint>
   <!-- Greifer-TCP (mittig zwischen den Fingerspitzen, grob). -->

Commit message: Hang the measured gripper model on the arm without moving the TCP

File: rg6/src/rg6_description/urdf/clearpath_extras.urdf.xacro (robot description, xacro)
@@ -40,31 +40,39 @@
   </joint>
   <!-- ===================== RG6-Greifer an arm_0_tool0 =================== -->
-  <!-- Greifermodell instanziieren (Praefix 'rg6_'). -->
-  <xacro:include filename="$(find rg6_description)/urdf/onrobot_rg6_model_macro.xacro"/>
-  <xacro:onrobot_rg6 prefix="rg6_"/>
-  <!-- Greiferbasis an den Tool-Flansch. Modell-Achse = +Z (wie altes Modell),
-       daher Roll -90deg um X. Falls noch verdreht, je 90deg variieren:
-         rpy="1.5708 0 0" | rpy="0 0 1.5708" | rpy="0 0 -1.5708"
-       z = 0: der Greifer sitzt UNMITTELBAR auf dem Flansch.  Am 2026-08-19
-       vom Owner am Geraet nachgesehen, nachdem hier zwischenzeitlich 0,0196
-       stand.  Diese 19,6 mm kamen aus ROBOTER-TODO R20, das aus dem
-       QC-Datenblatt geschlossen hatte, die ROBOTERSEITE des Quick Changers
-       fehle im Modell.  Der Schluss setzte eine separate QC-Scheibe zwischen
-       Flansch und Greifer voraus; die gibt es an diesem Roboter nicht.  Der
-       Fuss der Greiferbasis IST die Kopplungsflaeche (Ø71 mm, am Mesh
-       gemessen; unterste 20 mm von base_link.stl, und im fremden rg6_v2-Modell
-       ebenso als unterste Scheibe des single_bracket) und schraubt direkt auf
-       den Flansch.  Dazwischen liegt nur der 0,4-mm-Zentrierring des
-       UR-Flansches, und der ist eine Vertiefung, kein Aufbau. -->
-  <joint name="rg6_tool0_to_base" type="fixed">
-    <parent link="arm_0_tool0"/>
-    <child link="rg6_onrobot_rg6_base_link"/>
+  <!-- Modell aus onrobot_description (rg6_v2, MIT, INRIA), einvendort;
+       Herkunft und Aenderungen in ../../../LICENSE-THIRD-PARTY.md.
+       KEIN Montageversatz: das single_bracket schraubt unmittelbar auf den
+       UR-Flansch (2026-08-19 am Geraet nachgesehen).  Sein Fuss IST die
+       Kopplungsflaeche, 71 mm Durchmesser.  Dazwischen liegt nur der
+       0,4-mm-Zentrierring des Flansches, und der ist eine Vertiefung.
+       driver_joint haelt den Namen fest, den der ganze Workspace kennt:
+       rg6_finger_joint, 0 = offen, positiv = zu.  Die Folgegelenke haengen
+       per mimic daran. -->
+  <xacro:include filename="$(find rg6_description)/urdf/onrobot_rg_upstream.urdf.xacro"/>
+  <xacro:onrobot_rg parent="arm_0_tool0" prefix="rg6_" model="rg6_v2"
+                    driver_joint="rg6_finger_joint">
     <origin xyz="0 0 0" rpy="0 0 -1.5708"/>
+  </xacro:onrobot_rg>
+  <!-- Alter Name, gleicher Ort.  rg6_onrobot_rg6_base_link ist der Bezugspunkt
+       des SRDF-Patches und der MuJoCo-Szenen; ihn hier zu erhalten kostet einen
+       leeren Link und spart eine Umbenennung in drei Repos. -->
+  <link name="rg6_onrobot_rg6_base_link"/>
+  <joint name="rg6_base_link_alias" type="fixed">
+    <parent link="rg6_gripper_body"/><child link="rg6_onrobot_rg6_base_link"/>
+    <origin xyz="0 0 0" rpy="0 0 0"/>
   </joint>
-  <!-- Greifer-TCP (mittig zwischen den Fingerspitzen, grob). -->
+  <!-- Greifer-TCP.  DERSELBE physische Punkt wie im alten Modell: 210 mm ueber
+       der Kopplungsflaeche, am Anfang der Padflaeche.  Das neue Modell setzt
+       seinen grasp_frame 58,1 mm weiter vorn (nahe dem Pad-ENDE); ihn zu
+       uebernehmen haette den TCP still verschoben und jede kalibrierte Groesse
+       entwertet (descend_offset, floor_height, camera_xy_offset).  Am
+       2026-08-19 bewusst so entschieden; wohin der TCP physikalisch gehoert,
+       ist eine eigene Frage (ROBOTER-TODO R19/R23).
+       Ausgedrueckt gegen grasp_frame, damit er an der Modellgeometrie haengt
+       und nicht wieder an einer freien Zahl. -->
   <link name="rg6_hand_tcp"/>
   <joint name="rg6_hand_tcp_joint" type="fixed">
-    <origin xyz="0 0 0.21" rpy="0 0 0"/>
-    <parent link="rg6_onrobot_rg6_base_link"/><child link="rg6_hand_tcp"/>
+    <parent link="rg6_gripper_grasp_frame"/><child link="rg6_hand_tcp"/>
+    <origin xyz="0 0 -0.0581" rpy="0 0 0"/>
   </joint>
   <!-- ===== Custom Top-Assembly (ersetzt a200.sensor_arch) ===== -->

Commit message: Drop the rotation that belonged to the mesh we replaced

File: rg6/src/rg6_description/urdf/clearpath_extras.urdf.xacro (robot description, xacro)
@@ -48,9 +48,18 @@
        driver_joint haelt den Namen fest, den der ganze Workspace kennt:
        rg6_finger_joint, 0 = offen, positiv = zu.  Die Folgegelenke haengen
-       per mimic daran. -->
+       per mimic daran.
+       KEINE Drehung.  Das ALTE Modell brauchte hier rpy="0 0 -1.5708", und
+       sein Kommentar sagte selbst, das sei erprobt ("falls noch verdreht, je
+       90 Grad variieren").  Diese Zahl gehoerte zu jenem Mesh; mitgeschleppt
+       stand der Greifer am 2026-08-19 sichtbar um 90 Grad verdreht.
+       Nachgemessen als Oeffnungsrichtung der Finger im Flanschrahmen:
+         altes Modell, rpy 0 0 -1.5708 -> [-1  0  0]   (so sah es korrekt aus)
+         neues Modell, rpy 0 0  0      -> [-1  0  0]   deckungsgleich
+         neues Modell, rpy 0 0 -1.5708 -> [ 0 +1  0]   die 90 Grad
+       Wer hier wieder eine Drehung eintragen will, misst vorher nach. -->
   <xacro:include filename="$(find rg6_description)/urdf/onrobot_rg_upstream.urdf.xacro"/>
   <xacro:onrobot_rg parent="arm_0_tool0" prefix="rg6_" model="rg6_v2"
                     driver_joint="rg6_finger_joint">
-    <origin xyz="0 0 0" rpy="0 0 -1.5708"/>
+    <origin xyz="0 0 0" rpy="0 0 0"/>
   </xacro:onrobot_rg>
   <!-- Alter Name, gleicher Ort.  rg6_onrobot_rg6_base_link ist der Bezugspunkt

Commit message: Keep the camera where it was by pinning the legacy link to the flange

File: rg6/src/rg6_description/urdf/clearpath_extras.urdf.xacro (robot description, xacro)
@@ -57,17 +57,29 @@
          neues Modell, rpy 0 0  0      -> [-1  0  0]   deckungsgleich
          neues Modell, rpy 0 0 -1.5708 -> [ 0 +1  0]   die 90 Grad
-       Wer hier wieder eine Drehung eintragen will, misst vorher nach. -->
+       Die Oeffnungsachse allein entscheidet das NICHT: sie ist eine Gerade,
+       [-1 0 0] und [+1 0 0] sind dieselbe, und welcher Finger im jeweiligen
+       Modell "1" heisst, ist willkuerlich.  0 und 180 Grad sind daran also
+       nicht unterscheidbar.  Der Owner hat am 2026-08-19 gesehen, dass ohne
+       Drehung 180 Grad fehlen; daher pi.  Wer es genauer will, misst an einem
+       UNSYMMETRISCHEN Merkmal (Kabelausgang, Sicherheitsschalter). -->
   <xacro:include filename="$(find rg6_description)/urdf/onrobot_rg_upstream.urdf.xacro"/>
   <xacro:onrobot_rg parent="arm_0_tool0" prefix="rg6_" model="rg6_v2"
                     driver_joint="rg6_finger_joint">
-    <origin xyz="0 0 0" rpy="0 0 0"/>
+    <origin xyz="0 0 0" rpy="0 0 3.14159"/>
   </xacro:onrobot_rg>
-  <!-- Alter Name, gleicher Ort.  rg6_onrobot_rg6_base_link ist der Bezugspunkt
-       des SRDF-Patches und der MuJoCo-Szenen; ihn hier zu erhalten kostet einen
-       leeren Link und spart eine Umbenennung in drei Repos. -->
+  <!-- Alter Name, GENAU alter Ort.  rg6_onrobot_rg6_base_link ist mehr als ein
+       Bezugspunkt fuer SRDF-Patch und MuJoCo-Szenen: die robot.yaml haengt die
+       KAMERA daran (camera_0_joint, xyz 0,023/0/0,125, rpy 0/-1,5708/-3,14).
+       Alles, was diesen Link verschiebt oder dreht, verschiebt die Kamera mit.
+       Erste Fassung haengte ihn an rg6_gripper_body; das sitzt 56,1 mm ueber
+       dem Flansch, die Kamera stand damit 56 mm zu hoch UND mitgedreht.  Er
+       haengt deshalb direkt an arm_0_tool0 und reproduziert exakt das alte
+       rg6_tool0_to_base: Ursprung am Flansch, rpy 0 0 -1,5708.  Damit ist er
+       vom Greifermodell ENTKOPPELT; wie dessen Mesh gedreht wird, ist eine
+       andere Frage und darf die Kamera nicht mehr anfassen. -->
   <link name="rg6_onrobot_rg6_base_link"/>
   <joint name="rg6_base_link_alias" type="fixed">
-    <parent link="rg6_gripper_body"/><child link="rg6_onrobot_rg6_base_link"/>
-    <origin xyz="0 0 0" rpy="0 0 0"/>
+    <parent link="arm_0_tool0"/><child link="rg6_onrobot_rg6_base_link"/>
+    <origin xyz="0 0 0" rpy="0 0 -1.5708"/>
   </joint>
   <!-- Greifer-TCP.  DERSELBE physische Punkt wie im alten Modell: 210 mm ueber

Commit message: Give the sensor arch a collision model, so move_group can no longer plan through it
husky_top_assembly carried only <visual>: visible in the viewer, absent for
collision checking, so a trajectory could pass through the arch without the
planner or check_state_validity noticing. It stands 0.772 m from the arm base
and the UR5 reaches 0.85 m.

Not a bounding box. The mesh fills its hull to 2.4 percent, so one box would
have walled off the whole rear of the robot and blocked legitimate motions.
Six boxes follow the decoded structure instead - two portal legs, cross member,
sensor head, two feet with the diagonal brace - 5.87 L against 91.3 L, and all
4560 mesh vertices fall inside them.

The boxes start 2 mm above the foot. The link origin sits exactly on the top
plate's upper face, and MoveIt reads a touch as a permanent collision, which
would have made every state invalid. Checked against the robot's loaded
robot_description: zero permanent overlaps.

The front bumper deliberately gets nothing: measured, it lies entirely inside
base_link's lower collision box, so it is redundant rather than unmodelled.

File: rg6/src/rg6_description/urdf/clearpath_extras.urdf.xacro (robot description, xacro)
@@ -109,4 +109,51 @@
       </geometry>
     </visual>
+    <!-- KOLLISION (ROBOTER-TODO R15).  Bis 2026-08-20 hatte dieser Link NUR
+         <visual>: im Viewer sichtbar, fuer move_group nicht vorhanden.  Eine
+         Bahn konnte durch den Buegel fuehren, ohne dass Planer oder
+         check_state_validity es bemerkt haetten.  Der Buegel steht 0,772 m von
+         der Armbasis, der UR5 reicht 0,85 m - er ist erreichbar.
+         KEINE Gesamt-Bounding-Box.  Das Mesh fuellt seine Huelle nur zu 2,4 %
+         aus (2,3 L Struktur in 91,3 L Huelle); eine einzelne Box haette das
+         ganze Heck zugemauert und legitime Bahnen blockiert.  Stattdessen
+         sechs Kaesten entlang der tatsaechlichen Struktur - zwei Portalbeine,
+         Quertraeger, Sensorkopf, zwei Fuesse mit Diagonalstrebe: zusammen
+         5,87 L.  Nachgerechnet: ALLE 4560 Mesh-Vertices liegen darin.
+         Die Kaesten stehen im MESH-Frame, deshalb tragen sie dieselbe
+         rpy="0 0 -1.5708" wie das <visual> oben.  Wer eine Zahl aendert, aendert
+         sie im Mesh-Frame und dreht sie NICHT von Hand mit.
+         2 mm ueber dem Fuss abgeschnitten (z beginnt bei 0,002 statt 0,000).
+         Der Link-Ursprung sitzt bei Welt-z 0,2307 - exakt auf der Oberkante
+         von top_plate_link (0,2240..0,2307).  Bei z=0 beruehren sich beide
+         Koerper, und MoveIt liest eine Beruehrung als DAUERKOLLISION: der
+         Roboter waere in jeder Stellung ungueltig, move_group haette nichts
+         mehr geplant.  Die 2 mm sind kein Modellverlust - dort steht die
+         Deckplatte, die selbst Kollisionsgeometrie hat.  Alternative waere ein
+         disable_collisions-Eintrag in der SRDF gewesen; die wird generiert,
+         der Schnitt hier haelt die Aenderung in EINER Datei. -->
+    <collision>  <!-- Portalbein links -->
+      <origin xyz="0.0500 -0.0475 0.2510" rpy="0 0 -1.5708"/>
+      <geometry><box size="0.035 0.030 0.498"/></geometry>
+    </collision>
+    <collision>  <!-- Portalbein rechts -->
+      <origin xyz="0.0500 -0.5725 0.2510" rpy="0 0 -1.5708"/>
+      <geometry><box size="0.035 0.030 0.498"/></geometry>
+    </collision>
+    <collision>  <!-- Quertraeger oben -->
+      <origin xyz="0.0500 -0.3100 0.4900" rpy="0 0 -1.5708"/>
+      <geometry><box size="0.560 0.030 0.050"/></geometry>
+    </collision>
+    <collision>  <!-- Sensorkopf -->
+      <origin xyz="0.0500 -0.3150 0.5500" rpy="0 0 -1.5708"/>
+      <geometry><box size="0.120 0.120 0.100"/></geometry>
+    </collision>
+    <collision>  <!-- Fuss links, inkl. Diagonalstrebe -->
+      <origin xyz="0.1500 -0.0475 0.0810" rpy="0 0 -1.5708"/>
+      <geometry><box size="0.035 0.230 0.158"/></geometry>
+    </collision>
+    <collision>  <!-- Fuss rechts, inkl. Diagonalstrebe -->
+      <origin xyz="0.1500 -0.5725 0.0810" rpy="0 0 -1.5708"/>
+      <geometry><box size="0.035 0.230 0.158"/></geometry>
+    </collision>
   </link>
   <joint name="husky_top_assembly_joint" type="fixed">
