Commit message: Let the caller name the driver joint so the wire keeps the name it has

File: rg6/src/rg6_description/urdf/onrobot_rg_upstream.urdf.xacro (robot description, xacro)
@@ -5,6 +5,14 @@
   <!-- onrobot gripper -->
   <xacro:macro name="onrobot_rg" params="parent *origin prefix:=''
-    model:='rg2_v1' safety_shield:=False bracket:='single_bracket' mount_angle:=0.0 standalone:=false real_hardware:=false">
+    model:='rg2_v1' safety_shield:=False bracket:='single_bracket' mount_angle:=0.0 standalone:=false real_hardware:=false
+    driver_joint:=''">
     <xacro:property name="gripper_name" value="${prefix}gripper"/>
+    <!-- Name des Treibergelenks.  Upstream heisst es "<prefix>gripper_joint";
+         dieser Workspace kennt seit jeher "rg6_finger_joint", und der Name
+         steht in /joint_states, im Profil, im SRDF-Patch, in der
+         Greiferbruecke und in den MuJoCo-Szenen.  Ein Parameter hier spart
+         eine Umbenennung auf dem Draht.  Leer = Upstream-Voreinstellung. -->
+    <xacro:property name="driver"
+                    value="${driver_joint if driver_joint else gripper_name + '_joint'}"/>
     <!-- load config from file -->
     <xacro:property name="config_file" value="$(find rg6_description)/config/${model}.yaml"/>
@@ -104,5 +112,5 @@
         <xacro:_inertial id="moment_arm"/>
       </link>
-      <joint name="${gripper_name + ('' if is_master else '_mirror')}_joint" type="revolute">
+      <joint name="${driver if is_master else driver + '_mirror'}" type="revolute">
         <parent link="${name}_origin"/>
         <child link = "${name}_moment_arm"/>
@@ -112,5 +120,5 @@
         <dynamics damping="0.17"/>
         <xacro:unless value="${is_master}">
-          <mimic joint="${gripper_name}_joint" multiplier="1" offset="0"/>
+          <mimic joint="${driver}" multiplier="1" offset="0"/>
         </xacro:unless>
       </joint>
@@ -136,5 +144,5 @@
         <xacro:_frame id="truss_arm" rpy="0.0 ${offset} 0.0"/>
         <xacro:_limit/>
-        <mimic joint="${gripper_name}_joint" multiplier="1" offset="0"/>
+        <mimic joint="${driver}" multiplier="1" offset="0"/>
       </joint>
       <!-- safety shield -->
@@ -161,5 +169,5 @@
           <xacro:_frame id="safety_shield" rpy="0.0 ${offset} 0.0"/>
           <xacro:_limit/>
-          <mimic joint="${gripper_name}_joint" multiplier="1" offset="0"/>
+          <mimic joint="${driver}" multiplier="1" offset="0"/>
         </joint>
       </xacro:if>
@@ -190,5 +198,5 @@
         <xacro:_frame id="finger_tip" rpy="0.0 ${-offset} 0.0"/>
         <xacro:_limit/>
-        <mimic joint="${gripper_name}_joint" multiplier="1" offset="0"/>
+        <mimic joint="${driver}" multiplier="1" offset="0"/>
       </joint>
       <!-- flex finger -->

Commit message: Address the meshes by package so Foxglove is allowed to serve them

File: rg6/src/rg6_description/urdf/onrobot_rg_upstream.urdf.xacro (robot description, xacro)
@@ -1,3 +1,11 @@
 <?xml version="1.0"?>
+<!-- Meshpfade: package:// statt des Upstream-"file://$(find ...)".
+     Zwei Gruende, beide gemessen am 2026-08-19:
+     1. Die foxglove_bridge liefert nur aus, was ihre asset_uri_allowlist
+        erlaubt, und die lautet "^package://...".  Mit file:// zeigt Foxglove
+        das Modell OHNE Meshes; genau das war das Symptom am Roboter.
+     2. file://$(find ...) nagelt den absoluten Pfad des BAUENDEN Rechners
+        ins Modell (/home/robot/onrobot-rg6/install/...).  Weder Workstation
+        noch Container noch eine Wiedergabe koennen ihn aufloesen. -->
 <robot xmlns:xacro="http://wiki.ros.org/xacro" name="onrobot_rg_macro">
   <!-- materials -->
@@ -40,5 +48,5 @@
       <visual>
         <geometry>
-          <mesh filename="file://$(find rg6_description)/meshes/${model}/visual/${bracket}.stl"/>
+          <mesh filename="package://rg6_description/meshes/${model}/visual/${bracket}.stl"/>
         </geometry>
         <material name="onrobot/grey"/>
@@ -46,5 +54,5 @@
       <collision>
         <geometry>
-          <mesh filename="file://$(find rg6_description)/meshes/${model}/collision/${bracket}.stl"/>
+          <mesh filename="package://rg6_description/meshes/${model}/collision/${bracket}.stl"/>
         </geometry>
       </collision>
@@ -60,5 +68,5 @@
       <visual>
         <geometry>
-          <mesh filename="file://$(find rg6_description)/meshes/${model}/visual/body.stl"/>
+          <mesh filename="package://rg6_description/meshes/${model}/visual/body.stl"/>
         </geometry>
         <material name="onrobot/light_grey"/>
@@ -66,5 +74,5 @@
       <collision>
         <geometry>
-          <mesh filename="file://$(find rg6_description)/meshes/${model}/collision/body.stl"/>
+          <mesh filename="package://rg6_description/meshes/${model}/collision/body.stl"/>
         </geometry>
       </collision>
@@ -101,5 +109,5 @@
         <visual>
           <geometry>
-            <mesh filename="file://$(find rg6_description)/meshes/${model}/visual/moment_arm.stl"/>
+            <mesh filename="package://rg6_description/meshes/${model}/visual/moment_arm.stl"/>
           </geometry>
           <material name="onrobot/light_grey"/>
@@ -107,5 +115,5 @@
         <collision>
           <geometry>
-            <mesh filename="file://$(find rg6_description)/meshes/${model}/collision/moment_arm.stl"/>
+            <mesh filename="package://rg6_description/meshes/${model}/collision/moment_arm.stl"/>
           </geometry>
         </collision>
@@ -127,5 +135,5 @@
         <visual>
           <geometry>
-            <mesh filename="file://$(find rg6_description)/meshes/${model}/visual/truss_arm.stl"/>
+            <mesh filename="package://rg6_description/meshes/${model}/visual/truss_arm.stl"/>
           </geometry>
           <material name="onrobot/light_grey"/>
@@ -133,5 +141,5 @@
         <collision>
           <geometry>
-            <mesh filename="file://$(find rg6_description)/meshes/${model}/collision/truss_arm.stl"/>
+            <mesh filename="package://rg6_description/meshes/${model}/collision/truss_arm.stl"/>
           </geometry>
         </collision>
@@ -151,5 +159,5 @@
           <visual>
             <geometry>
-              <mesh filename="file://$(find rg6_description)/meshes/${model}/visual/safety_shield.stl"/>
+              <mesh filename="package://rg6_description/meshes/${model}/visual/safety_shield.stl"/>
             </geometry>
             <material name="onrobot/dark_grey"/>
@@ -157,5 +165,5 @@
           <collision>
             <geometry>
-              <mesh filename="file://$(find rg6_description)/meshes/${model}/collision/safety_shield.stl"/>
+              <mesh filename="package://rg6_description/meshes/${model}/collision/safety_shield.stl"/>
               <box size="0.0 0.0 0.0"/>
             </geometry>
@@ -176,5 +184,5 @@
         <visual>
           <geometry>
-            <mesh filename="file://$(find rg6_description)/meshes/${model}/visual/finger_tip.stl"/>
+            <mesh filename="package://rg6_description/meshes/${model}/visual/finger_tip.stl"/>
           </geometry>
           <material name="onrobot/light_grey"/>
@@ -182,10 +190,10 @@
         <collision>
           <geometry>
-            <mesh filename="file://$(find rg6_description)/meshes/${model}/visual/finger_tip.stl"/>
-          </geometry>
-        </collision>
-        <collision>
-          <geometry>
-            <mesh filename="file://$(find rg6_description)/meshes/${model}/visual/finger_tip.stl"/>
+            <mesh filename="package://rg6_description/meshes/${model}/visual/finger_tip.stl"/>
+          </geometry>
+        </collision>
+        <collision>
+          <geometry>
+            <mesh filename="package://rg6_description/meshes/${model}/visual/finger_tip.stl"/>
           </geometry>
         </collision>
@@ -204,5 +212,5 @@
         <visual>
           <geometry>
-            <mesh filename="file://$(find rg6_description)/meshes/${model}/visual/flex_finger.stl"/>
+            <mesh filename="package://rg6_description/meshes/${model}/visual/flex_finger.stl"/>
           </geometry>
           <material name="onrobot/dark_grey"/>
@@ -210,5 +218,5 @@
         <collision>
           <geometry>
-            <mesh filename="file://$(find rg6_description)/meshes/${model}/collision/flex_finger.stl"/>
+            <mesh filename="package://rg6_description/meshes/${model}/collision/flex_finger.stl"/>
           </geometry>
         </collision>

Commit message: Give the finger tip one collision mesh instead of the same one twice

File: rg6/src/rg6_description/urdf/onrobot_rg_upstream.urdf.xacro (robot description, xacro)
@@ -188,9 +188,8 @@
           <material name="onrobot/light_grey"/>
         </visual>
-        <collision>
-          <geometry>
-            <mesh filename="package://rg6_description/meshes/${model}/visual/finger_tip.stl"/>
-          </geometry>
-        </collision>
+        <!-- EINE Kollision, nicht zwei.  Upstream fuehrt diesen Block doppelt;
+             im kompilierten MuJoCo-Modell erschien der finger_tip dadurch mit
+             zwei identischen Kollisionsmeshes (2026-08-19 gemessen).  Das
+             kostet Kollisionspruefungen und bringt nichts. -->
         <collision>
           <geometry>

Commit message: fix(rg6_description): give the finger tip the collision meshes the package ships
Every other link resolves its collision geometry out of meshes/*/collision;
the finger tip alone pointed at the visual mesh -- and that is the gripping
surface.  Measured 2026-08-28: the visual mesh is 2154 triangles and concave,
so any engine that convexifies inflates it to 2.04x its volume, while the two
supplied parts are already convex (hull/mesh = 1.00) at 236 and 176 triangles.
They are a decomposition, which is why there are two of them and why the tip
now carries two collision elements rather than one.

File: rg6/src/rg6_description/urdf/onrobot_rg_upstream.urdf.xacro (robot description, xacro)
@@ -188,11 +188,20 @@
           <material name="onrobot/light_grey"/>
         </visual>
-        <!-- EINE Kollision, nicht zwei.  Upstream fuehrt diesen Block doppelt;
-             im kompilierten MuJoCo-Modell erschien der finger_tip dadurch mit
-             zwei identischen Kollisionsmeshes (2026-08-19 gemessen).  Das
-             kostet Kollisionspruefungen und bringt nichts. -->
-        <collision>
-          <geometry>
-            <mesh filename="package://rg6_description/meshes/${model}/visual/finger_tip.stl"/>
+        <!-- ZWEI Kollisionen, und zwar die dafuer gelieferten: die Spitze ist als konvexe
+             Zerlegung modelliert (finger_tip_1 und finger_tip_2), waehrend jedes andere Glied
+             hier ohnehin sein collision/-Mesh benutzt.  Upstream zeigt an dieser einen Stelle
+             auf das SICHTNETZ, und das ist die Greifflaeche: 2154 Dreiecke, konkav, und jede
+             Engine, die konvexifiziert, blaeht sie auf das 2,04-fache ihres Volumens auf
+             (2026-08-28 gemessen).  Die beiden Kollisionsteile sind bereits konvex
+             (Huelle/Netz = 1,00) und zusammen 236 + 176 Dreiecke.  Upstream fuehrte den Block
+             doppelt, aber mit demselben Sichtnetz -- daher die Zerlegung statt einer Kopie. -->
+        <collision>
+          <geometry>
+            <mesh filename="package://rg6_description/meshes/${model}/collision/finger_tip_1.stl"/>
+          </geometry>
+        </collision>
+        <collision>
+          <geometry>
+            <mesh filename="package://rg6_description/meshes/${model}/collision/finger_tip_2.stl"/>
           </geometry>
         </collision>

Commit message: feat(rg6_description): derive mass and inertia from the collision meshes
Upstream shipped one placeholder for every part, mass 0.001 with
ixx = iyy = izz = 0.001: three orders too light for a hand the data sheet puts
at 1.25 kg, about four orders too stiff for a part that fits in 3 cm. The whole
model weighed 0.789 kg, so 0.461 kg were missing from the wrist of the UR5.

The new tools/derive_link_inertia.py integrates each collision mesh exactly
(Eberly, polyhedral mass properties), gives the parts one homogeneous density
and fixes it so the sum over all instances is the data sheet's 1.25 kg. The
density comes out at 1343.1 kg/m^3.

Cross-checked against the second data sheet figure, which nothing in the
derivation aims at: the centre of gravity lands 90.58 mm above the tool base
point against the published 90.0 mm. That also settles a reading the mass alone
leaves open, namely that the 1.25 kg includes the mounting bracket.

The _inertial macro now writes an <origin> as well: without it URDF reads a
tensor taken about the part's centre of mass as being about the link frame,
which for the body is 52 mm out, and it parses either way.

File: rg6/src/rg6_description/urdf/onrobot_rg_upstream.urdf.xacro (robot description, xacro)
@@ -37,6 +37,11 @@
       <origin xyz="${origin[id]['x']} ${origin[id]['y']} ${origin[id]['z']}" rpy="${rpy}"/>
     </xacro:macro>
+    <!-- The <origin> is what makes the tensor mean anything: it is taken about the part's own centre of mass, and
+         without the offset URDF reads it as being about the LINK frame instead.  For the body that is 52 mm out,
+         and the error goes into the model as a mass that hangs in the wrong place rather than as a parse failure.
+         rpy stays zero, because the tensor is written in the link's axes and not in its principal ones. -->
     <xacro:macro name="_inertial" params="id">
       <inertial>
+        <origin xyz="${inertial[id]['cx']} ${inertial[id]['cy']} ${inertial[id]['cz']}" rpy="0 0 0"/>
         <mass value="${inertial[id]['mass']}"/>
         <inertia ixx="${inertial[id]['ixx']}" iyy="${inertial[id]['iyy']}" izz="${inertial[id]['izz']}"
