Commit message: refactor(extras): make the rg6 and key holder tools parent-parametric macros
rg6.macro.xacro and key_holder.macro.xacro hang each tool on a given parent.
The a200 tool files call them on arm_0_tool0 and keep the camera alias; the
expanded links and joints are identical to before. The file tests now cover
every xacro under src/.

File: extras/src/husky_extras_description/urdf/tools/key_holder.urdf.xacro (robot description, xacro)
@@ -1,12 +1,5 @@
 <?xml version="1.0"?>
 <!--
-  A printed key holder on the UR5's flange (ISO 9409-1-50, 63 mm) carrying a Rittal double-bit key, for opening
-  control cabinets: end_effector:=key_holder.  Meshes from mujoco-mia (scenes/endeffector), in the holder frame:
-  +z out of the flange, the holder 0..50 mm, the key's tip at 107.8 mm, its bit across y.
-  The meshes are drawn; primitives collide, sized off the meshes (2026-09-22): the holder a cylinder, the shank a thin
-  cylinder, the bit a box 16 x 4 x 6 mm.  The holder is turned half a turn on the flange, with the camera clamped to it;
-  holder and key are point-symmetric about the flange axis (the key within 3 mm), so only the camera shows it.  key_tip
-  is the tool's TCP: the point that enters a lock, with the flange's axes.  The key holder has no joints: nothing
-  drives it, so the offboard mock starts no gripper for it.
+  The key holder (key_holder.macro.xacro) on the UR5's flange, for opening control cabinets: end_effector:=key_holder.
   rg6_onrobot_rg6_base_link keeps the name robot.yaml hangs the wrist camera on, and stands where that puts the camera
   on THIS tool: on the RG6 the D435 sits 136 mm out along the flange axis, past this key's tip, and would meet a door
@@ -17,40 +10,6 @@
 -->
 <robot xmlns:xacro="http://ros.org/wiki/xacro">
-  <link name="key_holder">
-    <inertial>
-      <origin xyz="0 0 0.04" rpy="0 0 0"/>
-      <mass value="0.12"/>
-      <inertia ixx="8e-5" iyy="8e-5" izz="5e-5" ixy="0" ixz="0" iyz="0"/>
-    </inertial>
-    <visual>
-      <geometry><mesh filename="package://husky_extras_description/meshes/key_holder/key_holder.obj"/></geometry>
-      <material name="key_holder_blue"><color rgba="0.6157 0.8118 0.9294 1"/></material>
-    </visual>
-    <visual>
-      <geometry><mesh filename="package://husky_extras_description/meshes/key_holder/key.obj"/></geometry>
-      <material name="key_metal"><color rgba="0.62 0.62 0.6 1"/></material>
-    </visual>
-    <collision>  <!-- holder -->
-      <origin xyz="0 0 0.025" rpy="0 0 0"/>
-      <geometry><cylinder radius="0.0315" length="0.05"/></geometry>
-    </collision>
-    <collision>  <!-- shank -->
-      <origin xyz="0 0 0.0745" rpy="0 0 0"/>
-      <geometry><cylinder radius="0.003" length="0.049"/></geometry>
-    </collision>
-    <collision>  <!-- bit: passes a 10 x 22 mm keyhole upright, is caught across it -->
-      <origin xyz="0 0 0.1048" rpy="0 0 0"/>
-      <geometry><box size="0.004 0.016 0.006"/></geometry>
-    </collision>
-  </link>
-  <joint name="key_holder_joint" type="fixed">
-    <parent link="arm_0_tool0"/><child link="key_holder"/>
-    <origin xyz="0 0 0" rpy="0 0 3.14159"/>
-  </joint>
-  <link name="key_tip"/>
-  <joint name="key_tip_joint" type="fixed">
-    <parent link="arm_0_tool0"/><child link="key_tip"/>
-    <origin xyz="0 0 0.1078" rpy="0 0 0"/>
-  </joint>
+  <xacro:include filename="../key_holder.macro.xacro"/>
+  <xacro:key_holder parent="arm_0_tool0"/>
   <link name="rg6_onrobot_rg6_base_link"/>
   <joint name="rg6_base_link_alias" type="fixed">

File: extras/src/husky_extras_description/urdf/tools/rg6.urdf.xacro (robot description, xacro)
@@ -17,36 +17,6 @@
 -->
 <robot xmlns:xacro="http://ros.org/wiki/xacro">
-  <!-- ===================== RG6 gripper at arm_0_tool0 =================== -->
-  <!-- The model itself is vendored in the OTHER repo: rg6_description
-       (onrobot-rg6) carries the meshes, the macro and the measured rg6_v2.yaml,
-       and its LICENSE-THIRD-PARTY.md carries origin and changes of the
-       onrobot_description model (rg6_v2, MIT, INRIA).  What stands here is only
-       where the hand is bolted on.
-       NO mounting offset: the single_bracket screws straight onto the UR
-       flange (looked at on the device on 2026-08-19).  Its foot IS the coupling
-       face, 71 mm in diameter.  Between them lies only the 0.4 mm centring ring
-       of the flange, and that is a recess.
-       driver_joint pins the name the whole workspace knows:
-       rg6_finger_joint, 0 = open, positive = closed.  The dependent joints hang
-       on it by mimic.
-       NO rotation.  The OLD model needed rpy="0 0 -1.5708" here, and its own
-       comment said that was found by trial ("if still twisted, vary in steps of
-       90 degrees").  That number belonged to that mesh; carried over, the
-       gripper stood visibly twisted by 90 degrees on 2026-08-19.  Measured as
-       the opening direction of the fingers in the flange frame:
-         old model, rpy 0 0 -1.5708 -> [-1  0  0]   (this is how it looked right)
-         new model, rpy 0 0  0      -> [-1  0  0]   congruent
-         new model, rpy 0 0 -1.5708 -> [ 0 +1  0]   the 90 degrees
-       The opening axis alone does NOT decide this: it is a straight line,
-       [-1 0 0] and [+1 0 0] are the same one, and which finger is called "1" in
-       either model is arbitrary.  0 and 180 degrees are therefore not
-       distinguishable by it.  The owner saw on 2026-08-19 that 180 degrees are
-       missing without the rotation; hence pi.  Whoever wants it more precisely
-       measures at an ASYMMETRIC feature (cable outlet, safety switch). -->
-  <xacro:include filename="$(find rg6_description)/urdf/onrobot_rg_upstream.urdf.xacro"/>
-  <xacro:onrobot_rg parent="arm_0_tool0" prefix="rg6_" model="rg6_v2"
-                    driver_joint="rg6_finger_joint">
-    <origin xyz="0 0 0" rpy="0 0 3.14159"/>
-  </xacro:onrobot_rg>
+  <xacro:include filename="../rg6.macro.xacro"/>
+  <xacro:rg6_tool parent="arm_0_tool0"/>
   <!-- The old name, EXACTLY the old place.  rg6_onrobot_rg6_base_link is more
        than a reference point for the SRDF patch and the MuJoCo scenes: robot.yaml
@@ -65,17 +35,3 @@
     <origin xyz="0 0 0" rpy="0 0 -1.5708"/>
   </joint>
-  <!-- Gripper TCP.  THE SAME physical point as in the old model: 210 mm above
-       the coupling face, at the start of the pad surface.  The new model puts its
-       grasp_frame 58.1 mm further forward (near the END of the pad); taking that
-       over would have moved the TCP silently and devalued every calibrated
-       quantity (descend_offset, floor_height, camera_xy_offset).  Deliberately
-       decided that way on 2026-08-19; where the TCP physically belongs is a
-       question of its own (ROBOTER-TODO R19/R23).
-       Expressed against grasp_frame, so that it hangs on the model geometry and
-       not on a free number again. -->
-  <link name="rg6_hand_tcp"/>
-  <joint name="rg6_hand_tcp_joint" type="fixed">
-    <parent link="rg6_gripper_grasp_frame"/><child link="rg6_hand_tcp"/>
-    <origin xyz="0 0 -0.0581" rpy="0 0 0"/>
-  </joint>
 </robot>
