Commit message: feat(extras): select the end effector with the end_effector argument
clearpath_extras.urdf.xacro includes urdf/tools/<end_effector>.urdf.xacro,
default rg6, which robot.yaml leaves as it is. The RG6 block moved unchanged
into tools/rg6.urdf.xacro. tools/key_holder.urdf.xacro adds the Rittal key
holder of the cabinet task: meshes from mujoco-mia, primitive collisions, TCP
key_tip, and the wrist camera clamped to the holder on the flange's +y side,
upright; the holder sits half a turn on the flange (R61: placed, not measured).
The tests read every tool file.

File: extras/src/husky_extras_description/urdf/clearpath_extras.urdf.xacro (robot description, xacro)
@@ -8,5 +8,5 @@
             path: /home/robot/husky-extras/src/husky_extras_description/urdf/clearpath_extras.urdf.xacro
   Hangs ONLY new links/joints onto frames the generator has already produced:
-    - arm_0_tool0         = UR5 tool frame (ROS-Industrial all-zeros)  -> RG6 gripper
+    - arm_0_tool0         = UR5 tool frame (ROS-Industrial all-zeros)  -> the end effector (tools/, RG6 by default)
     - top_plate_rear_mount = frame the sensor arch stands on
     - top_plate_front_mount = frame the ArUco marker sits on (TODO: adjust)
@@ -17,14 +17,5 @@
   dependency therefore runs one way only: this package includes
   rg6_description's macro, and rg6_description includes nothing from here.
-  GRIPPER MODEL:
-    A cleanly articulated RG6 from package 'rg6_description' (Robotiq style:
-    outer_knuckle/inner_knuckle/inner_finger per side). Driver joint =
-    'rg6_finger_joint' (prefix 'rg6_'): 0 = open, positive = closed. The 5
-    dependent joints hang on the driver joint via <mimic> (the official OnRobot
-    multipliers) -> MoveIt animates them in the planning preview, the ROS 2
-    robot_state_publisher computes them for /tf (Foxglove). The
-    rg6_joint_state_broadcaster additionally publishes all 6 joints explicitly
-    (fallback / live tuning of the AI2 mapping); the values match <mimic>.
-    Collision = one coarse box at the base_link (no self-collision in MoveIt).
+  END EFFECTOR: tools/<end_effector>.urdf.xacro; tools/rg6.urdf.xacro says how the RG6 is modelled.
   PRECONDITION: BOTH packages have to be installed in a workspace listed in
   robot.yaml under 'system.ros2.workspaces': 'husky_extras_description' for
@@ -53,66 +44,10 @@
     <origin rpy="0 0 0" xyz="-0.062 -0.142 0"/>  <!-- R48: unverified offset -->
   </joint>
-  <!-- ===================== RG6 gripper at arm_0_tool0 =================== -->
-  <!-- The model itself is vendored in the OTHER repo: rg6_description
-       (onrobot-rg6) carries the meshes, the macro and the measured rg6_v2.yaml,
-       and its LICENSE-THIRD-PARTY.md carries origin and changes of the
-       onrobot_description model (rg6_v2, MIT, INRIA).  What stands here is only
-       where the hand is bolted on.
-       NO mounting offset: the single_bracket screws straight onto the UR
-       flange (looked at on the device on 2026-08-19).  Its foot IS the coupling
-       face, 71 mm in diameter.  Between them lies only the 0.4 mm centring ring
-       of the flange, and that is a recess.
-       driver_joint pins the name the whole workspace knows:
-       rg6_finger_joint, 0 = open, positive = closed.  The dependent joints hang
-       on it by mimic.
-       NO rotation.  The OLD model needed rpy="0 0 -1.5708" here, and its own
-       comment said that was found by trial ("if still twisted, vary in steps of
-       90 degrees").  That number belonged to that mesh; carried over, the
-       gripper stood visibly twisted by 90 degrees on 2026-08-19.  Measured as
-       the opening direction of the fingers in the flange frame:
-         old model, rpy 0 0 -1.5708 -> [-1  0  0]   (this is how it looked right)
-         new model, rpy 0 0  0      -> [-1  0  0]   congruent
-         new model, rpy 0 0 -1.5708 -> [ 0 +1  0]   the 90 degrees
-       The opening axis alone does NOT decide this: it is a straight line,
-       [-1 0 0] and [+1 0 0] are the same one, and which finger is called "1" in
-       either model is arbitrary.  0 and 180 degrees are therefore not
-       distinguishable by it.  The owner saw on 2026-08-19 that 180 degrees are
-       missing without the rotation; hence pi.  Whoever wants it more precisely
-       measures at an ASYMMETRIC feature (cable outlet, safety switch). -->
-  <xacro:include filename="$(find rg6_description)/urdf/onrobot_rg_upstream.urdf.xacro"/>
-  <xacro:onrobot_rg parent="arm_0_tool0" prefix="rg6_" model="rg6_v2"
-                    driver_joint="rg6_finger_joint">
-    <origin xyz="0 0 0" rpy="0 0 3.14159"/>
-  </xacro:onrobot_rg>
-  <!-- The old name, EXACTLY the old place.  rg6_onrobot_rg6_base_link is more
-       than a reference point for the SRDF patch and the MuJoCo scenes: robot.yaml
-       hangs the CAMERA on it (camera_0_joint, xyz 0.023/0/0.125,
-       rpy 0/-1.5708/-3.14).  Everything that moves or turns this link moves the
-       camera with it.
-       The first version hung it on rg6_gripper_body; that sits 56.1 mm above the
-       flange, which put the camera 56 mm too high AND turned along.  It therefore
-       hangs directly on arm_0_tool0 and reproduces the old rg6_tool0_to_base
-       exactly: origin at the flange, rpy 0 0 -1.5708.  That DECOUPLES it from the
-       gripper model; how the latter's mesh is turned is a separate question and
-       must not touch the camera any more. -->
-  <link name="rg6_onrobot_rg6_base_link"/>
-  <joint name="rg6_base_link_alias" type="fixed">
-    <parent link="arm_0_tool0"/><child link="rg6_onrobot_rg6_base_link"/>
-    <origin xyz="0 0 0" rpy="0 0 -1.5708"/>
-  </joint>
-  <!-- Gripper TCP.  THE SAME physical point as in the old model: 210 mm above
-       the coupling face, at the start of the pad surface.  The new model puts its
-       grasp_frame 58.1 mm further forward (near the END of the pad); taking that
-       over would have moved the TCP silently and devalued every calibrated
-       quantity (descend_offset, floor_height, camera_xy_offset).  Deliberately
-       decided that way on 2026-08-19; where the TCP physically belongs is a
-       question of its own (ROBOTER-TODO R19/R23).
-       Expressed against grasp_frame, so that it hangs on the model geometry and
-       not on a free number again. -->
-  <link name="rg6_hand_tcp"/>
-  <joint name="rg6_hand_tcp_joint" type="fixed">
-    <parent link="rg6_gripper_grasp_frame"/><child link="rg6_hand_tcp"/>
-    <origin xyz="0 0 -0.0581" rpy="0 0 0"/>
-  </joint>
+  <!-- ======================= end effector at arm_0_tool0 ======================= -->
+  <!-- One file per tool under tools/, chosen by end_effector (rg6 when nothing is said, as on the robot); the
+       offboard mock passes end_effector:=<name> (the tool option of up.sh).  A path relative to this file rather than
+       $(find ...): the generator reads this file from the source tree, and the tool files stand beside it there. -->
+  <xacro:arg name="end_effector" default="rg6"/>
+  <xacro:include filename="tools/$(arg end_effector).urdf.xacro"/>
   <!-- ===== custom top assembly (replaces a200.sensor_arch) ===== -->
   <link name="husky_top_assembly">

Commit message: docs(extras): shorten the URDF mounting comments to their measurements and constraints

File: extras/src/husky_extras_description/urdf/clearpath_extras.urdf.xacro (robot description, xacro)
@@ -52,18 +52,7 @@
   <!-- ===== custom top assembly (replaces a200.sensor_arch) ===== -->
   <link name="husky_top_assembly">
-    <!-- INERTIAL.  Until now this link had collision geometry and no mass at all, and that is not the harmless
-         omission it looks like: `twinlink.urdf_mujoco._ensure_inertial` substitutes 0.1 kg for any link without
-         one, so both simulators have been carrying a half-metre portal frame as a tenth of a kilogram.
-         The volume is measured, the density is assumed, and the two are worth different amounts of trust.  2.3 L of
-         structure is R15's own figure from the mesh (2026-08-20, quoted in the collision comment below); 2700 kg/m^3
-         is the textbook density of the 6xxx aluminium profile the arch is built from, and NOT a measurement on this
-         arch.  2.3 L at that density is 6.21 kg.  Weighing it closes the assumption (R47).  The tensor distributes
-         the mass over the six collision boxes by volume, which is likewise not the true distribution but is one
-         anybody can recompute, with the box mode of tools/derive_link_inertia.py:
-             python3 ../onrobot-rg6/tools/derive_link_inertia.py (box-link mode)
-                 ../husky-extras/src/husky_extras_description/urdf/clearpath_extras.urdf.xacro \
-                 husky_top_assembly 6.21
-         What this is NOT good enough for is a claim about how the Husky tips; for that the arch goes on a scale.
-         What it IS good enough for is not lying to the simulator by a factor of 62. -->
+    <!-- R47: mass is estimated, not weighed: mesh volume 2.3 L (2026-08-20) at an assumed aluminum density
+         of 2700 kg/m^3 gives 6.21 kg. The inertia distributes this mass over the six collision boxes by volume;
+         recompute with onboard/rg6/tools/derive_link_inertia.py. Do not use it to claim tipping stability. -->
     <inertial>
       <origin xyz="0.093339 -0.311227 0.284882" rpy="0 0 0"/>
@@ -82,27 +71,9 @@
       </geometry>
     </visual>
-    <!-- COLLISION (ROBOTER-TODO R15).  Until 2026-08-20 this link had ONLY a
-         <visual>: visible in the viewer, non-existent for move_group.  A path
-         could lead straight through the arch without the planner or
-         check_state_validity noticing.  The arch stands 0.772 m from the arm
-         base, the UR5 reaches 0.85 m - it is reachable.
-         NO overall bounding box.  The mesh fills its hull to only 2.4 %
-         (2.3 L of structure in a 91.3 L hull); a single box would have walled up
-         the whole rear and blocked legitimate paths.  Instead six boxes along the
-         actual structure - two portal legs, cross beam, sensor head, two feet
-         with a diagonal strut: 5.87 L together.  Recomputed: ALL 4560 mesh
-         vertices lie inside them.
-         The boxes stand in the MESH frame, which is why they carry the same
-         rpy="0 0 -1.5708" as the <visual> above.  Whoever changes a number
-         changes it in the mesh frame and does NOT rotate it by hand.
-         Cut off 2 mm above the foot (z starts at 0.002 instead of 0.000).  The
-         link origin sits at world z 0.2307 - exactly on the upper edge of
-         top_plate_link (0.2240..0.2307).  At z=0 the two bodies touch, and MoveIt
-         reads a touch as a PERMANENT COLLISION: the robot would be invalid in
-         every pose, and move_group would have planned nothing at all.  The 2 mm
-         are no loss of model - the top plate stands there, and it carries
-         collision geometry of its own.  The alternative would have been a
-         disable_collisions entry in the SRDF; that one is generated, and the cut
-         here keeps the change in ONE file. -->
+    <!-- R15 (2026-08-20): the arch is reachable (0.772 m from the arm base, UR5 reach 0.85 m).
+         Six boxes enclose all 4560 mesh vertices in 5.87 L; one hull box would obstruct the open portal
+         (2.3 L of structure in a 91.3 L hull). Coordinates remain in the mesh frame, with the visual's rotation.
+         The feet start 2 mm above top_plate_link: its upper surface and this link's origin are both at
+         world z=0.2307 m, and touching would make every MoveIt state invalid. The plate covers that gap. -->
     <collision>  <!-- portal leg, left -->
       <origin xyz="0.0500 -0.0475 0.2510" rpy="0 0 -1.5708"/>

File: extras/src/husky_extras_description/urdf/rg6.macro.xacro (robot description, xacro)
@@ -8,30 +8,8 @@
   <xacro:macro name="rg6_tool" params="parent">
     <!-- ===================== RG6 gripper at ${parent} ===================== -->
-    <!-- The model itself is vendored in the OTHER repo: rg6_description
-         (onrobot-rg6) carries the meshes, the macro and the measured rg6_v2.yaml,
-         and its LICENSE-THIRD-PARTY.md carries origin and changes of the
-         onrobot_description model (rg6_v2, MIT, INRIA).  What stands here is only
-         where the hand is bolted on.
-         NO mounting offset: the single_bracket screws straight onto the UR
-         flange (looked at on the device on 2026-08-19).  Its foot IS the coupling
-         face, 71 mm in diameter.  Between them lies only the 0.4 mm centring ring
-         of the flange, and that is a recess.
-         driver_joint pins the name the whole workspace knows:
-         rg6_finger_joint, 0 = open, positive = closed.  The dependent joints hang
-         on it by mimic.
-         NO rotation.  The OLD model needed rpy="0 0 -1.5708" here, and its own
-         comment said that was found by trial ("if still twisted, vary in steps of
-         90 degrees").  That number belonged to that mesh; carried over, the
-         gripper stood visibly twisted by 90 degrees on 2026-08-19.  Measured as
-         the opening direction of the fingers in the flange frame:
-           old model, rpy 0 0 -1.5708 -> [-1  0  0]   (this is how it looked right)
-           new model, rpy 0 0  0      -> [-1  0  0]   congruent
-           new model, rpy 0 0 -1.5708 -> [ 0 +1  0]   the 90 degrees
-         The opening axis alone does NOT decide this: it is a straight line,
-         [-1 0 0] and [+1 0 0] are the same one, and which finger is called "1" in
-         either model is arbitrary.  0 and 180 degrees are therefore not
-         distinguishable by it.  The owner saw on 2026-08-19 that 180 degrees are
-         missing without the rotation; hence pi.  Whoever wants it more precisely
-         measures at an ASYMMETRIC feature (cable outlet, safety switch). -->
+    <!-- The bracket sits directly on the flange, with no mounting offset (observed 2026-08-19).
+         The owner confirmed the half-turn on that date; the opening axis alone cannot distinguish 0 from pi.
+         Refine the rotation against an asymmetric feature such as the cable outlet.
+         rg6_finger_joint is 0 when open and positive when closed; dependent joints use mimic. -->
     <xacro:include filename="$(find rg6_description)/urdf/onrobot_rg_upstream.urdf.xacro"/>
     <xacro:onrobot_rg parent="${parent}" prefix="rg6_" model="rg6_v2"
@@ -39,13 +17,6 @@
       <origin xyz="0 0 0" rpy="0 0 3.14159"/>
     </xacro:onrobot_rg>
-    <!-- Gripper TCP.  THE SAME physical point as in the old model: 210 mm above
-         the coupling face, at the start of the pad surface.  The new model puts its
-         grasp_frame 58.1 mm further forward (near the END of the pad); taking that
-         over would have moved the TCP silently and devalued every calibrated
-         quantity (descend_offset, floor_height, camera_xy_offset).  Deliberately
-         decided that way on 2026-08-19; where the TCP physically belongs is a
-         question of its own (ROBOTER-TODO R19/R23).
-         Expressed against grasp_frame, so that it hangs on the model geometry and
-         not on a free number again. -->
+    <!-- R19/R23: the calibrated TCP is 210 mm above the flange, at the start of the pads;
+         grasp_frame is 58.1 mm farther out (2026-08-19). Changing this offset invalidates TCP calibrations. -->
     <link name="rg6_hand_tcp"/>
     <joint name="rg6_hand_tcp_joint" type="fixed">

File: extras/src/husky_extras_description/urdf/tools/rg6.urdf.xacro (robot description, xacro)
@@ -19,15 +19,6 @@
   <xacro:include filename="../rg6.macro.xacro"/>
   <xacro:rg6_tool parent="arm_0_tool0"/>
-  <!-- The old name, EXACTLY the old place.  rg6_onrobot_rg6_base_link is more
-       than a reference point for the SRDF patch and the MuJoCo scenes: robot.yaml
-       hangs the CAMERA on it (camera_0_joint, xyz 0.023/0/0.125,
-       rpy 0/-1.5708/-3.14).  Everything that moves or turns this link moves the
-       camera with it.
-       The first version hung it on rg6_gripper_body; that sits 56.1 mm above the
-       flange, which put the camera 56 mm too high AND turned along.  It therefore
-       hangs directly on arm_0_tool0 and reproduces the old rg6_tool0_to_base
-       exactly: origin at the flange, rpy 0 0 -1.5708.  That DECOUPLES it from the
-       gripper model; how the latter's mesh is turned is a separate question and
-       must not touch the camera any more. -->
+  <!-- robot.yaml mounts the camera on this frame. Keep it directly on the flange so changes to the
+       gripper mesh or body frame cannot move the calibrated camera mount. -->
   <link name="rg6_onrobot_rg6_base_link"/>
   <joint name="rg6_base_link_alias" type="fixed">

Commit message: feat(extras)!: remove the ArUco marker from the a200-0553's URDF
The marker hung on top_plate_front_mount at an offset that was placed, never surveyed (R48); nothing in the stack addresses it, and a frame nobody measured misleads any pose estimation that trusts it. The extras carry the sensor arch and the end effector only; a test holds the marker out.

BREAKING CHANGE: the links aruco_marker and aruco_to_base are gone from robot_description once the extras are rolled out.

File: extras/src/husky_extras_description/urdf/clearpath_extras.urdf.xacro (robot description, xacro)
@@ -10,5 +10,4 @@
     - arm_0_tool0         = UR5 tool frame (ROS-Industrial all-zeros)  -> the end effector (tools/, RG6 by default)
     - top_plate_rear_mount = frame the sensor arch stands on
-    - top_plate_front_mount = frame the ArUco marker sits on (TODO: adjust)
   WHY THIS IS ITS OWN PACKAGE.  Everything here is THIS ROBOT's assembly, not a
   component: it names frames that only exist once the Clearpath generator has
@@ -26,22 +25,4 @@
 -->
 <robot xmlns:xacro="http://ros.org/wiki/xacro">
-  <material name="white"><color rgba="0.9137 0.9137 0.9137 1.0"/></material>
-  <!-- =========================== ArUco marker =========================== -->
-  <!-- R48: neither the parent frame nor the offset has been measured on the
-       robot.  Both numbers below are placed, not surveyed, and the marker is
-       visual only (no collision, no mass), so nothing plans against it; what it
-       misleads is a human reading the viewer, and any pose estimation that
-       trusts the frame. -->
-  <link name="aruco_marker">
-    <visual>
-      <geometry><box size="0.11 0.11 0.001"/></geometry>
-      <material name="white"/>
-    </visual>
-  </link>
-  <joint name="aruco_to_base" type="fixed">
-    <parent link="top_plate_front_mount"/>          <!-- R48: unverified frame -->
-    <child link="aruco_marker"/>
-    <origin rpy="0 0 0" xyz="-0.062 -0.142 0"/>  <!-- R48: unverified offset -->
-  </joint>
   <!-- ======================= end effector at arm_0_tool0 ======================= -->
   <!-- One file per tool under tools/, chosen by end_effector (rg6 when nothing is said, as on the robot); the
